Commit message: feat(urdf): make the ros2_control command interface selectable
Adds a command_interface argument (default: effort, so existing setups
are unaffected) to leg.xacro, unitree_go2_robot.xacro and the simulation
launch file. This allows driving the robot through the position
interface without editing the description by hand.

File: unitree_go2_description/urdf/leg.xacro (robot description, xacro)
@@ -2,5 +2,6 @@
 <robot xmlns:xacro="http://www.ros.org/wiki/xacro">
     <!-- <xacro:include filename="$(find unitree_go2_description)/transmission.xacro"/> -->
-    <xacro:macro name="leg" params="name mirror mirror_dae front_hind front_hind_dae">
+    <xacro:macro name="leg"
+        params="name mirror mirror_dae front_hind front_hind_dae command_interface:=effort">
         <joint name="${name}_hip_joint" type="revolute">
             <xacro:if value="${(mirror_dae == False) and (front_hind_dae == True)}">
@@ -160,15 +161,15 @@
             </hardware>
             <joint name="${name}_hip_joint">
-                <command_interface name="effort"/>
+                <command_interface name="${command_interface}"/>
                 <state_interface name="position"/>
                 <state_interface name="velocity"/>
             </joint>
             <joint name="${name}_upper_leg_joint">
-                <command_interface name="effort"/>
+                <command_interface name="${command_interface}"/>
                 <state_interface name="position"/>
                 <state_interface name="velocity"/>
             </joint>
             <joint name="${name}_lower_leg_joint">
-                <command_interface name="effort"/>
+                <command_interface name="${command_interface}"/>
                 <state_interface name="position"/>
                 <state_interface name="velocity"/>

File: unitree_go2_description/urdf/unitree_go2_robot.xacro (robot description, xacro)
@@ -4,4 +4,6 @@
     <xacro:arg name="DEBUG" default="false"/>
     <xacro:arg name="robot_controllers" default="$(find unitree_go2_sim)/config/ros_control/ros_control.yaml"/>
+    <!-- Joint command interface used by ros2_control: "effort" or "position" -->
+    <xacro:arg name="command_interface" default="effort"/>
     <xacro:include filename="$(find unitree_go2_description)/urdf/const.xacro" />
     <xacro:include filename="$(find unitree_go2_description)/urdf/materials.xacro" />
@@ -171,7 +173,11 @@
         </collision>
     </link> -->
-    <xacro:leg name="rf" mirror="-1" mirror_dae="False" front_hind="1" front_hind_dae="True" />
-    <xacro:leg name="lf" mirror="1" mirror_dae="True" front_hind="1" front_hind_dae="True" />
-    <xacro:leg name="rh" mirror="-1" mirror_dae="False" front_hind="-1" front_hind_dae="False" />
-    <xacro:leg name="lh" mirror="1" mirror_dae="True" front_hind="-1" front_hind_dae="False" />
+    <xacro:leg name="rf" mirror="-1" mirror_dae="False" front_hind="1" front_hind_dae="True"
+        command_interface="$(arg command_interface)" />
+    <xacro:leg name="lf" mirror="1" mirror_dae="True" front_hind="1" front_hind_dae="True"
+        command_interface="$(arg command_interface)" />
+    <xacro:leg name="rh" mirror="-1" mirror_dae="False" front_hind="-1" front_hind_dae="False"
+        command_interface="$(arg command_interface)" />
+    <xacro:leg name="lh" mirror="1" mirror_dae="True" front_hind="-1" front_hind_dae="False"
+        command_interface="$(arg command_interface)" />
 </robot>
