Commit message: feat(gazebo): publish foot contacts from the simulated feet
Adds a contact sensor to each foot link, loads the gz contact system in
the default world, and bridges the four topics to ROS as
ros_gz_interfaces/msg/Contacts.

Two supporting changes were needed:

- preserveFixedJoint on the foot joints. Without it Gazebo lumps the
foot link into the lower leg, the collision named in the sensor no
longer exists and the sensor stays silent
- self_collide is dropped on the foot links. With self collision enabled
the feet report contacts against the robot's own links, which the sensor
cannot distinguish from ground contact

File: unitree_go2_description/urdf/unitree_go2_gazebo.xacro (robot description, xacro)
@@ -183,7 +183,19 @@
             <mu1>0.6</mu1>
             <mu2>0.6</mu2>
-            <self_collide>1</self_collide>
-            <kp>10000.0</kp>
-            <kd>1.0</kd>
+            <kp>10000.0</kp>
+            <kd>1.0</kd>
+            <sensor name="lf_foot_contact_sensor" type="contact">
+                <always_on>true</always_on>
+                <update_rate>100.0</update_rate>
+                <contact>
+                    <collision>lf_foot_link_collision</collision>
+                    <topic>/lf_foot_contacts</topic>
+                </contact>
+            </sensor>
+        </gazebo>
+        <!-- Keep the fixed foot joint, otherwise Gazebo lumps the foot link
+             into the lower leg and the contact sensor has no collision -->
+        <gazebo reference="lf_foot_joint">
+            <preserveFixedJoint>true</preserveFixedJoint>
         </gazebo>
         <!-- FR leg -->
@@ -207,7 +219,19 @@
             <mu1>0.6</mu1>
             <mu2>0.6</mu2>
-            <self_collide>1</self_collide>
-            <kp>10000.0</kp>
-            <kd>1.0</kd>
+            <kp>10000.0</kp>
+            <kd>1.0</kd>
+            <sensor name="rf_foot_contact_sensor" type="contact">
+                <always_on>true</always_on>
+                <update_rate>100.0</update_rate>
+                <contact>
+                    <collision>rf_foot_link_collision</collision>
+                    <topic>/rf_foot_contacts</topic>
+                </contact>
+            </sensor>
+        </gazebo>
+        <!-- Keep the fixed foot joint, otherwise Gazebo lumps the foot link
+             into the lower leg and the contact sensor has no collision -->
+        <gazebo reference="rf_foot_joint">
+            <preserveFixedJoint>true</preserveFixedJoint>
         </gazebo>
         <!-- RL leg -->
@@ -231,7 +255,19 @@
             <mu1>0.6</mu1>
             <mu2>0.6</mu2>
-            <self_collide>1</self_collide>
-            <kp>10000.0</kp>
-            <kd>1.0</kd>
+            <kp>10000.0</kp>
+            <kd>1.0</kd>
+            <sensor name="lh_foot_contact_sensor" type="contact">
+                <always_on>true</always_on>
+                <update_rate>100.0</update_rate>
+                <contact>
+                    <collision>lh_foot_link_collision</collision>
+                    <topic>/lh_foot_contacts</topic>
+                </contact>
+            </sensor>
+        </gazebo>
+        <!-- Keep the fixed foot joint, otherwise Gazebo lumps the foot link
+             into the lower leg and the contact sensor has no collision -->
+        <gazebo reference="lh_foot_joint">
+            <preserveFixedJoint>true</preserveFixedJoint>
         </gazebo>
   <!-- RR leg -->
@@ -255,8 +291,20 @@
     <mu1>0.6</mu1>
     <mu2>0.6</mu2>
-    <self_collide>1</self_collide>
     <kp>10000.0</kp>
     <kd>1.0</kd>
-  </gazebo>
+            <sensor name="rh_foot_contact_sensor" type="contact">
+                <always_on>true</always_on>
+                <update_rate>100.0</update_rate>
+                <contact>
+                    <collision>rh_foot_link_collision</collision>
+                    <topic>/rh_foot_contacts</topic>
+                </contact>
+            </sensor>
+        </gazebo>
+        <!-- Keep the fixed foot joint, otherwise Gazebo lumps the foot link
+             into the lower leg and the contact sensor has no collision -->
+        <gazebo reference="rh_foot_joint">
+            <preserveFixedJoint>true</preserveFixedJoint>
+        </gazebo>
 </xacro:macro>
 </robot>
